Commit message: prismatic gripper

File: urdf/owi535.urdf (robot description, URDF)
Before this commit: robot test_robot, 5 links, 4 joints
Links:
- removed link gripper
- added link gripper_base; visual mesh filename=package://owi535/meshes/gripper_base.dae
- added link gripper_left; visual mesh filename=package://owi535/meshes/gripper_left.dae
- added link gripper_right; visual mesh filename=package://owi535/meshes/gripper_right.dae
Joints:
- added joint wrist_left: type prismatic, parent gripper_base, child gripper_left, origin xyz=0 0 0 rpy=0.0 0 0, axis 0 1 0, limit lower=-4.00 upper=4.00 effort=3 velocity=1.178465545
- added joint wrist_right: type prismatic, parent gripper_base, child gripper_right, origin xyz=0 0 0 rpy=0.0 0 0, axis 0 1 0, limit lower=-4.00 upper=4.00 effort=3 velocity=1.178465545, mimic joint=wrist_left multiplier=-1.0
- joint wrist: child gripper -> gripper_base

Commit message: detailed the gripper

File: urdf/owi535.urdf (robot description, URDF)
Before this commit: robot test_robot, 7 links, 6 joints
Links:
- removed link gripper_base
- removed link gripper_left
- removed link gripper_right
- added link back; visual mesh filename=package://owi535/meshes/back.dae
- added link left_carpal; visual mesh filename=package://owi535/meshes/left_carpal.dae
- added link left_finger; visual mesh filename=package://owi535/meshes/right_finger_tip.dae
- added link left_phalange; visual mesh filename=package://owi535/meshes/phalange.dae
- added link right_carpal; visual mesh filename=package://owi535/meshes/right_carpal.dae
- added link right_finger; visual mesh filename=package://owi535/meshes/left_finger_tip.dae
- added link right_phalange; visual mesh filename=package://owi535/meshes/phalange.dae
- added link wrist_base; visual mesh filename=package://daru/meshes/wrist.dae
Joints:
- removed joint wrist_left
- removed joint wrist_right
- added joint left_f: type revolute, parent left_phalange, child left_finger, origin xyz=8.0 0 0 rpy=0 0 3.14, axis 0 0 1.0, limit lower=-0.08 upper=1.20 effort=3 velocity=1.178465545, mimic joint=left_grip multiplier=-1.0 offset=3.14
- added joint left_grip: type revolute, parent back, child left_carpal, origin xyz=14.7 4.0 0 rpy=3.14 0 0, axis 0 0 1.0, limit lower=-1.20 upper=-0.08 effort=3 velocity=1.178465545
- added joint left_ph: type revolute, parent back, child left_phalange, origin xyz=20.0 2.0 0 rpy=3.14 0 0, axis 0 0 1.0, limit lower=-0.08 upper=1.20 effort=3 velocity=1.178465545, mimic joint=left_grip multiplier=1.0
- added joint right_f: type revolute, parent right_phalange, child right_finger, origin xyz=8.0 0 0 rpy=0 0 3.14, axis 0 0 1.0, limit lower=-0.08 upper=1.20 effort=3 velocity=1.178465545, mimic joint=right_grip multiplier=-1.0 offset=3.14
- added joint right_grip: type revolute, parent back, child right_carpal, origin xyz=14.7 -4.0 0 rpy=3.14 0 0, axis 0 0 1.0, limit lower=-0.08 upper=1.20 effort=3 velocity=1.178465545, mimic joint=left_grip multiplier=-1.0
- added joint right_ph: type revolute, parent back, child right_phalange, origin xyz=20.0 -2.0 0 rpy=3.14 0 0, axis 0 0 1.0, limit lower=-0.08 upper=1.20 effort=3 velocity=1.178465545, mimic joint=left_grip multiplier=-1.0
- added joint wrist_base: type revolute, parent radius, child wrist_base, origin xyz=-50 0 0 rpy=0 0 3.14, axis 0 1.0 0, limit lower=-1.57 upper=1.57 effort=3 velocity=1.178465545
- joint wrist: axis 0 1 0 -> 0 1.0 0; child gripper_base -> back; origin xyz=-50 0 0 rpy=0 0 0 -> xyz=0 0 0 rpy=0 0 0; parent radius -> wrist_base

Commit message: added the shield

File: urdf/owi535.urdf (robot description, URDF)
Before this commit: robot test_robot, 12 links, 11 joints
Links:
- added link shield; visual mesh filename=package://owi535/meshes/shield.dae
Joints:
- added joint shield_fix: type fixed, parent back, child shield, origin xyz=0 0 0 rpy=0 0 3.14
- joint wrist_base: type revolute -> fixed

Commit message: gazebo files added as in the rrbot tutorial

File: urdf/owi535.urdf (robot description, URDF)
Before this commit: robot test_robot, 13 links, 12 joints
Links:
- added link camera_link, mass 1e-5; collision box size=15 10 5; visual box size=15 10 5
- link back: mass None -> 0.1
- link base: mass None -> 0.1; geometry collision box size=5 5 5; visual mesh filename=package://owi535/meshes/shoulder.dae
- link base_link: mass None -> 1; geometry collision box size=50 30 20; visual mesh filename=package://owi535/meshes/accupack.dae
- link humerus: mass None -> 0.1; geometry collision box size=15 5 5; visual mesh filename=package://owi535/meshes/humerus.dae
- link left_carpal: mass None -> 1e-5
- link left_finger: mass None -> 1e-5
- link radius: mass None -> 0.1; geometry collision box size=15 5 5; visual mesh filename=package://owi535/meshes/radius.dae
- link right_carpal: mass None -> 1e-5
- link right_finger: mass None -> 1e-5
- link right_phalange: mass None -> 1e-5
- link shield: mass None -> 0.1
- link wrist_base: mass None -> 0.1; geometry visual mesh filename=package://owi535/meshes/wrist.dae
Joints:
- added joint camera_joint: type fixed, parent back, child camera_link, origin xyz=0 0 0 rpy=0 0 3.14

Commit message: scaled down everything to the wrist

File: urdf/owi535.urdf (robot description, URDF)
Before this commit: robot test_robot, 14 links, 13 joints
Links:
- removed link back
- removed link base
- removed link camera_link
- removed link humerus
- removed link left_carpal
- removed link left_finger
- removed link left_phalange
- removed link radius
- removed link right_carpal
- removed link right_finger
- removed link right_phalange
- removed link shield
- added link elbow_motor, mass 0.1; collision box size=0.05 0.05 0.05; visual mesh filename=package://owi535/meshes/shoulder.dae
- added link humerus_left, mass 0.1; collision box size=15 5 5; visual mesh filename=package://owi535/meshes/humerus_link.dae
- added link humerus_right, mass 0.1; collision box size=15 5 5; visual mesh filename=package://owi535/meshes/humerus_link.dae
- added link radius_link_down, mass 0.1; collision box size=15 5 5; visual mesh filename=package://owi535/meshes/radius_link.dae
- added link radius_link_up, mass 0.1; collision box size=15 5 5; visual mesh filename=package://owi535/meshes/radius_link.dae
- added link rotation_base, mass 0.1; collision box size=0.05 0.05 0.05; visual mesh filename=package://owi535/meshes/rotation_base.dae
- added link shoulder_motor, mass 0.1; collision box size=0.05 0.05 0.05; visual mesh filename=package://owi535/meshes/shoulder.dae
- added link switchboard, mass 0.1; collision box size=0.05 0.05 0.05; visual mesh filename=package://owi535/meshes/switchboard.dae
- added link wrist_motor, mass 0.1; collision box size=0.05 0.05 0.05; visual mesh filename=package://owi535/meshes/shoulder.dae
- link base_link: geometry collision box size=0.05 0.030 0.020; visual mesh filename=package://owi535/meshes/battery_pack.dae
Joints:
- removed joint camera_joint
- removed joint left_f
- removed joint left_grip
- removed joint left_ph
- removed joint right_f
- removed joint right_grip
- removed joint right_ph
- removed joint shield_fix
- added joint humerus: type fixed, parent humerus_left, child humerus_right, origin xyz=0 -0.0466 0 rpy=0 0 3.14
- added joint lower_radius: type fixed, parent elbow_motor, child radius_link_down, origin xyz=0.01 0 -0.0155 rpy=0 0 0
- added joint rotator: type fixed, parent base_link, child rotation_base, origin xyz=0 0 0 rpy=0 0 0
- added joint switcher: type fixed, parent base_link, child switchboard, origin xyz=0.12 0 0.0500 rpy=0 0 0
- added joint upper_radius: type fixed, parent elbow_motor, child radius_link_up, origin xyz=0.01 0 0.0178 rpy=3.14 0 0
- joint elbow: child radius -> elbow_motor; origin xyz=0 0 50 rpy=0 0 0 -> xyz=0 -0.0233 0.1010 rpy=0 0 0; parent humerus -> humerus_left
- joint rotationbase: child base -> shoulder_motor; origin xyz=0 0 21 rpy=0 0 0 -> xyz=0 0 0.0580 rpy=0 0 0
- joint shoulder: child humerus -> humerus_left; origin xyz=0 0 7 rpy=0 0 0 -> xyz=0 0.0233 0 rpy=0 0 0; parent base -> shoulder_motor
- joint wrist: axis 0 1.0 0 -> (none); child back -> wrist_motor; limit lower=-1.57 upper=1.57 effort=3 velocity=1.178465545 -> (none); origin xyz=0 0 0 rpy=0 0 0 -> xyz=-0.0721 0 0 rpy=0 0 0; parent wrist_base -> elbow_motor; type revolute -> fixed
- joint wrist_base: axis 0 1.0 0 -> (none); limit lower=-1.57 upper=1.57 effort=3 velocity=1.178465545 -> (none); origin xyz=-50 0 0 rpy=0 0 3.14 -> xyz=-0.03 0 0 rpy=0 0 3.14; parent radius -> wrist_motor

Commit message: added the parts of the gripper to the model

File: urdf/owi535.urdf (robot description, URDF)
Before this commit: robot test_robot, 11 links, 10 joints
Links:
- added link back, mass 0.1; visual mesh filename=package://owi535/meshes/back.dae
- added link left_carpal, mass 1e-5; visual mesh filename=package://owi535/meshes/left_carpal.dae
- added link left_finger, mass 1e-5; visual mesh filename=package://owi535/meshes/right_finger_tip.dae
- added link left_phalange; visual mesh filename=package://owi535/meshes/phalange.dae
- added link right_carpal, mass 1e-5; visual mesh filename=package://owi535/meshes/right_carpal.dae
- added link right_finger, mass 1e-5; visual mesh filename=package://owi535/meshes/left_finger_tip.dae
- added link right_phalange, mass 1e-5; visual mesh filename=package://owi535/meshes/phalange.dae
- added link shield, mass 0.1; visual mesh filename=package://owi535/meshes/shield.dae
Joints:
- added joint left_f: type revolute, parent left_phalange, child left_finger, origin xyz=0.0234 0 0 rpy=0 0 3.14, axis 0 0 1.0, limit lower=-0.08 upper=1.20 effort=3 velocity=1.178465545, mimic joint=left_grip multiplier=-1.0 offset=3.14
- added joint left_grip: type revolute, parent back, child left_carpal, origin xyz=0.0416 0.0135 0 rpy=3.14 0 0, axis 0 0 1.0, limit lower=-1.20 upper=-0.08 effort=3 velocity=1.178465545
- added joint left_ph: type revolute, parent back, child left_phalange, origin xyz=0.05856 0.0065 0 rpy=3.14 0 0, axis 0 0 1.0, limit lower=-0.08 upper=1.20 effort=3 velocity=1.178465545, mimic joint=left_grip multiplier=1.0
- added joint right_f: type revolute, parent right_phalange, child right_finger, origin xyz=0.0234 0 0 rpy=0 0 3.14, axis 0 0 1.0, limit lower=-0.08 upper=1.20 effort=3 velocity=1.178465545, mimic joint=right_grip multiplier=-1.0 offset=3.14
- added joint right_grip: type revolute, parent back, child right_carpal, origin xyz=0.0416 -0.0135 0 rpy=3.14 0 0, axis 0 0 1.0, limit lower=-0.08 upper=1.20 effort=3 velocity=1.178465545, mimic joint=left_grip multiplier=-1.0
- added joint right_ph: type revolute, parent back, child right_phalange, origin xyz=0.05856 -0.0065 0 rpy=3.14 0 0, axis 0 0 1.0, limit lower=-0.08 upper=1.20 effort=3 velocity=1.178465545, mimic joint=left_grip multiplier=-1.0
- added joint shield_fix: type fixed, parent back, child shield, origin xyz=0 0 0 rpy=0 0 3.14
- added joint wrist_fixed: type fixed, parent elbow_motor, child wrist_motor, origin xyz=-0.0721 0 0 rpy=0 0 0
- joint wrist: axis (none) -> 0 1.0 0; child wrist_motor -> back; limit (none) -> lower=-1.57 upper=1.57 effort=3 velocity=1.178465545; origin xyz=-0.0721 0 0 rpy=0 0 0 -> xyz=0 0 0 rpy=0 0 0; parent elbow_motor -> wrist_base; type fixed -> revolute

Commit message: fingertip refactored, unused meshes removed

File: urdf/owi535.urdf (robot description, URDF)
Before this commit: robot test_robot, 19 links, 18 joints
Links:
- link elbow_motor: geometry collision box size=0.05 0.05 0.05; visual mesh filename=package://owi535/meshes/gearbox.dae
- link left_finger: geometry visual mesh filename=package://owi535/meshes/finger_tip_link.dae
- link right_finger: geometry visual mesh filename=package://owi535/meshes/finger_tip_link.dae
- link shoulder_motor: geometry collision box size=0.05 0.05 0.05; visual mesh filename=package://owi535/meshes/gearbox.dae
- link wrist_motor: geometry collision box size=0.05 0.05 0.05; visual mesh filename=package://owi535/meshes/gearbox.dae
Joints:
- joint left_f: origin xyz=0.0234 0 0 rpy=0 0 3.14 -> xyz=0.0234 0 0.009 rpy=0 0 3.14
- joint right_f: origin xyz=0.0234 0 0 rpy=0 0 3.14 -> xyz=0.0234 0 0.009 rpy=0 0 3.14

Commit message: added three markers to the gazebo scene + controllers to move the robot

File: urdf/owi535.urdf (robot description, URDF)
Before this commit: robot test_robot, 19 links, 18 joints
Links:
- added link battery_pack, mass 1; collision box size=0.22 0.114 0.043; visual mesh filename=package://owi535/meshes/battery_pack.dae
- link base_link: mass 1 -> None; geometry 
- link elbow_motor: geometry visual mesh filename=package://owi535/meshes/gearbox.dae
- link humerus_left: geometry visual mesh filename=package://owi535/meshes/humerus_link.dae
- link humerus_right: geometry visual mesh filename=package://owi535/meshes/humerus_link.dae
- link radius_link_down: geometry visual mesh filename=package://owi535/meshes/radius_link.dae
- link radius_link_up: geometry visual mesh filename=package://owi535/meshes/radius_link.dae
- link rotation_base: geometry visual mesh filename=package://owi535/meshes/rotation_base.dae
- link shoulder_motor: geometry visual mesh filename=package://owi535/meshes/gearbox.dae
- link switchboard: geometry visual mesh filename=package://owi535/meshes/switchboard.dae
- link wrist_motor: geometry visual mesh filename=package://owi535/meshes/gearbox.dae
Joints:
- added joint dummyjoint: type fixed, parent base_link, child battery_pack, origin xyz=0 0 0 rpy=0 0 0

Commit message: added gazebo camera

File: urdf/owi535.urdf (robot description, URDF)
Before this commit: robot test_robot, 20 links, 19 joints
Links:
- added link camera_link, mass 1e-5; collision box size=0.08 0.04 0.01; visual box size=0.08 0.04 0.01
Joints:
- added joint camera_joint: type fixed, parent back, child camera_link, origin xyz=0.04 0 -0.01 rpy=0 0 0

Commit message: fixed transmissions + world link added

File: urdf/owi535.urdf (robot description, URDF)
Before this commit: robot test_robot, 21 links, 20 joints
Links:
- added link world
- link left_phalange: mass None -> 1e-5
Joints:
- added joint fixed: type fixed, parent world, child base_link

Commit message: AR tag markers are detected and published to tf
and can be seen in rviz

File: urdf/owi535.urdf (robot description, URDF)
Before this commit: robot test_robot, 22 links, 21 joints
Links:
- removed link rotation_base
- removed link wrist_base
- added link camera_link_optical, mass 1e-5; visual box size=0.08 0.04 0.01
- added link rotation_base_link, mass 0.1; visual mesh filename=package://owi535/meshes/rotation_base.dae
- added link wrist_base_link, mass 0.1; visual mesh filename=package://owi535/meshes/wrist.dae
- link camera_link: mass 1e-5 -> None; geometry visual box size=0.08 0.04 0.01
Joints:
- added joint camera_optical_joint: type fixed, parent camera_link, child camera_link_optical, origin xyz=0 0 0 rpy=-1.570796325 0 -1.570796325
- joint camera_joint: origin xyz=0.04 0 -0.01 rpy=0 0 0 -> xyz=0 0 0 rpy=0 0 0
- joint rotationbase: parent base_link -> rotation_base_link
- joint rotator: child rotation_base -> rotation_base_link
- joint wrist: parent wrist_base -> wrist_base_link
- joint wrist_base: child wrist_base -> wrist_base_link
