Commit message: baby steps towards AR marker driven position

File: urdf/marker21.urdf (robot description, URDF)
Before this commit: robot test_marker, 1 links, 0 joints
Links:
- removed link base_link
- added link marker21, mass 0.001; collision box size=0.05 0.05 0.05; visual mesh filename=package://owi535/meshes/marker21.dae
- added link world
Joints:
- added joint fixed21: type fixed, parent world, child marker21, origin xyz=-0.5 -0.2 0.2 rpy=0 1.57 0

File: urdf/marker22.urdf (robot description, URDF)
Before this commit: robot test_marker, 1 links, 0 joints
Links:
- removed link base_link
- added link marker22, mass 0.001; collision box size=0.05 0.05 0.05; visual mesh filename=package://owi535/meshes/marker22.dae
- added link world
Joints:
- added joint fixed22: type fixed, parent world, child marker22, origin xyz=-0.5 0 0.3 rpy=0 1.57 0

File: urdf/marker23.urdf (robot description, URDF)
Before this commit: robot test_marker, 1 links, 0 joints
Links:
- removed link base_link
- added link marker23, mass 0.001; collision box size=0.05 0.05 0.05; visual mesh filename=package://owi535/meshes/marker23.dae
- added link world
Joints:
- added joint fixed23: type fixed, parent world, child marker23, origin xyz=-0.5 0.2 0.2 rpy=0 1.57 0

File: urdf/owi535.urdf (robot description, URDF)
Before this commit: robot test_robot, 23 links, 22 joints
Links:
- link camera_link: mass None -> 1e-5
- link camera_link_optical: geometry visual box size=0.02 0.04 0.01
